File: zongle.kicad_pcb (KiCad board)
At the start: 6 copper layers, 13.5 x 14.4 mm, 20 parts, among them U1 453-00059R

Commit message: changes version number  to 0.0.5
Other:
- board text added: "zongle@0.0.5"
- board text removed: "zongle@0.0.4"
Changed lines of the file:
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@@
 		(layer "Edge.Cuts")
 	)
-	(gr_text "zongle@0.0.4"
+	(gr_text "zongle@0.0.5"
 		(at 154.27 116.65 0)
 		(layer "B.SilkS")
@@
 			(justify left bottom mirror)
 		)
-		(render_cache "zongle@0.0.4" 0
+		(render_cache "zongle@0.0.5" 0
 			(polygon
 				(pts
@@
 			(polygon
 				(pts
-					(xy 149.387096 116.565) (xy 149.387096 116.463578) (xy 149.613021 116.463578) (xy 149.613021 116.336968)
-					(xy 149.42416 116.054349) (xy 149.326921 116.054349) (xy 149.529093 116.360049) (xy 149.529093 116.386611)
-					(xy 149.387096 116.386611) (xy 149.387096 116.271206) (xy 149.298955 116.271206) (xy 149.298955 116.565)
-				)
-			)
+					(xy 149.447241 116.571991) (xy 149.484545 116.569253) (xy 149.516266 116.561516) (xy 149.543346 116.549231)
+					(xy 149.566523 116.532485) (xy 149.585703 116.511284) (xy 149.599429 116.4868) (xy 149.60793 116.458384)
+					(xy 149.610915 116.425109) (xy 149.523476 116.425109) (xy 149.52105 116.445667) (xy 149.514164 116.462522)
+					(xy 149.502868 116.476523) (xy 149.488038 116.486904) (xy 149.469597 116.493418) (xy 149.446539 116.495757)
+					(xy 149.423514 116.493403) (xy 149.405342 116.486878) (xy 149.390943 116.476523) (xy 149.380144 116.462526)
+					(xy 149.373418 116.445028) (xy 149.371007 116.423003) (xy 149.371007 116.389419) (xy 149.373383 116.367368)
+					(xy 149.380004 116.34987) (xy 149.390607 116.3359) (xy 149.404782 116.325558) (xy 149.422818 116.319028)
+					(xy 149.445837 116.316666) (xy 149.593451 116.316666) (xy 149.593451 116.054349) (xy 149.302436 116.054349)
+					(xy 149.302436 116.133392) (xy 149.510897 116.133392) (xy 149.510195 116.239729) (xy 149.441654 116.239729)
+					(xy 149.403858 116.242505) (xy 149.37251 116.250264) (xy 149.346469 116.262445) (xy 149.324845 116.2789)
+					(xy 149.30731 116.299704) (xy 149.294509 116.324481) (xy 149.286438 116.354028) (xy 149.283568 116.389419)
+					(xy 149.283568 116.423003) (xy 149.286533 116.457075) (xy 149.294953 116.486024) (xy 149.308483 116.510809)
+					(xy 149.327288 116.532118) (xy 149.350136 116.548955) (xy 149.377167 116.561355) (xy 149.40919 116.569202)
+				)
+			)
